Commit message: Add raspicam link

File: src/arlobot/arlobot_description/urdf/arlo.urdf.xacro (robot description, xacro)
@@ -233,4 +233,30 @@
       </collision>
     </link>
+    <link name="raspicam">
+      <inertial>
+        <origin xyz="0 0 0"/>
+        <mass value="0.01" />
+        <inertia ixx="0.001" ixy="0.0" ixz="0.0"
+          iyy="0.001" iyz="0.0" izz="0.001" />
+      </inertial>
+      <visual>
+        <origin xyz="0 0 0" rpy="0 0 0" />
+        <geometry>
+          <cylinder radius="0.01" length = "0.005"/>
+        </geometry>
+        <material name ="Green" />
+      </visual>
+      <collision>
+        <origin xyz="0 0 0" rpy="0 0 0" />
+        <geometry>
+          <cylinder radius="0.01" length = "0.005"/>
+        </geometry>
+      </collision>
+    </link>
+    <joint name="raspicam_footprint" type="fixed">
+      <origin xyz="-0.083 0 0.386" rpy="3.1416 -1.5707 0"/>
+      <parent link="base_footprint"/>
+      <child link="raspicam" />
+    </joint>
     <!-- Fixed because we never rotate it anyway, it is just for show -->
     <!-- NOTE This may prevent gazebo from working with this model -->

Commit message: Update urdf

File: src/arlobot/arlobot_description/urdf/arlo.urdf.xacro (robot description, xacro)
@@ -255,5 +255,5 @@
     </link>
     <joint name="raspicam_footprint" type="fixed">
-      <origin xyz="-0.083 0 0.386" rpy="3.1416 -1.5707 0"/>
+      <origin xyz="-0.083 0 0.386" rpy="0 0 1.5708"/>
       <parent link="base_footprint"/>
       <child link="raspicam" />

Commit message: Update URDF

File: src/arlobot/arlobot_description/urdf/arlo.urdf.xacro (robot description, xacro)
@@ -255,5 +255,5 @@
     </link>
     <joint name="raspicam_footprint" type="fixed">
-      <origin xyz="-0.083 0 0.386" rpy="0 0 1.5708"/>
+      <origin xyz="-0.083 0 0.37" rpy="0 0 1.5708"/>
       <parent link="base_footprint"/>
       <child link="raspicam" />
